Commit message: Quadcopter: give global mass

File: roboschool/models_robot/quadcopter_description/urdf/quadcopter-v1.urdf (robot description, URDF)
Before this commit: robot quadcopter, 6 links, 5 joints
Links:
- link base_link: mass 0.0 -> 1.0

Commit message: Quadcopter: pretty up the UDRF a bit

File: roboschool/models_robot/quadcopter_description/urdf/quadcopter-v1.urdf (robot description, URDF)
Before this commit: robot quadcopter, 6 links, 5 joints
Links:
- link BL: geometry collision cylinder length=0.03 radius=0.10; visual cylinder length=0.03 radius=0.10
- link BR: geometry collision cylinder length=0.03 radius=0.10; visual cylinder length=0.03 radius=0.10
- link FL: geometry collision cylinder length=0.03 radius=0.10; visual cylinder length=0.03 radius=0.10
- link FR: geometry collision cylinder length=0.03 radius=0.10; visual cylinder length=0.03 radius=0.10
- link base_link: geometry 
- link center: geometry collision box size=0.2 0.1 0.04; visual box size=0.2 0.1 0.04
Joints:
- joint base_to_BL: parent center -> base_link
- joint base_to_BR: parent center -> base_link
- joint base_to_FL: parent center -> base_link
- joint base_to_FR: parent center -> base_link
